File: Controller/controller.kicad_sch (KiCad schematic)
At the start: 5 parts, among them SW1 SW_Push, SW2 SW_Push, SW3 SW_Push, U1 XIAO-RP2040-DIP, U2 COM-09032

Commit message: Day 2 of controller
Parts:
- added D1: SK6812MINI, LED_SMD:LED_SK6812MINI_PLCC4_3.5x3.5mm_P1.75mm, symbol LED:SK6812MINI
- added U3: COM-09032, COM-09032:XDCR_COM-09032, symbol COM-09032:COM-09032
- SW1, SW2, SW3: footprint (none) -> Button_Switch_Keyboard:SW_Cherry_MX_1.00u_PCB
- U1: footprint Module:MOUDLE14P-XIAO-DIP-SMD -> Seeed Studio XIAO Series Library:XIAO-RP2040-DIP
Connections:
- net +5V: now also U2.H1 (H+), D1.4 (VDD), U3.H1 (H+), U3.V1 (V+)
- net GND: now also U2.H3 (H-), D1.2 (VSS), U3.B1A (SEL+), U3.B2A (SEL-), U3.H3 (H-), U3.S1 (SHIELD), U3.S2 (SHIELD), U3.S3 (SHIELD), U3.S4 (SHIELD), U3.V3 (V-)
- net at U1.2 (GPIO27/ADC1/A1): now also U2.V2 (V); no longer U2.H1 (H+)
- net at U2.H2 (H): now also U1.1 (GPIO26/ADC0/A0)
- net at U1.3 (GPIO28/ADC2/A2): now also U3.V2 (V)
- net at U1.4 (GPIO29/ADC3/A3): now also U3.H2 (H)
- net at U1.5 (GPIO6/SDA): now also D1.3 (DIN)

Commit message: (I think) I finished the firmware for the controller
Parts:
- added SW4: SW_Push, Button_Switch_Keyboard:SW_Cherry_MX_1.00u_PCB, symbol Switch:SW_Push
Connections:
- net GND: now also SW4.1
- net at U1.8 (GPIO1/RX): now also SW4.2
Other:
- moved on the sheet: SW1
Changed lines of the file:
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@@
 		(color 0 0 0 0)
 	)
+	(junction
+		(at 101.6 62.23)
+		(diameter 0)
+		(color 0 0 0 0)
+	)
 	(wire
 		(pts
@@
 	(wire
 		(pts
+			(xy 163.83 167.64) (xy 163.83 93.98)
+		)
+		(stroke
+			(width 0)
+			(type default)
+		)
+	)
+	(wire
+		(pts
+			(xy 111.76 90.17) (xy 111.76 114.3)
+		)
+		(stroke
+			(width 0)
+			(type default)
+		)
+	)
+	(wire
+		(pts
+			(xy 81.28 167.64) (xy 163.83 167.64)
+		)
+		(stroke
+			(width 0)
+			(type default)
+		)
+	)
+	(wire
+		(pts
 			(xy 115.57 74.93) (xy 115.57 111.76)
 		)
@@
 	(wire
 		(pts
+			(xy 101.6 62.23) (xy 101.6 74.93)
+		)
+		(stroke
+			(width 0)
+			(type default)
+		)
+	)
+	(wire
+		(pts
 			(xy 172.72 92.71) (xy 172.72 107.95)
 		)
@@
 	(wire
 		(pts
-			(xy 111.76 90.17) (xy 111.76 114.3)
+			(xy 113.03 60.96) (xy 121.92 60.96)
 		)
 		(stroke
@@
 	(wire
 		(pts
+			(xy 69.85 153.67) (xy 81.28 153.67)
+		)
+		(stroke
+			(width 0)
+			(type default)
+		)
+	)
+	(wire
+		(pts
 			(xy 180.34 82.55) (xy 163.83 82.55)
 		)
@@
 	(wire
 		(pts
+			(xy 111.76 74.93) (xy 115.57 74.93)
+		)
+		(stroke
+			(width 0)
+			(type default)
+		)
+	)
+	(wire
+		(pts
+			(xy 111.76 114.3) (xy 180.34 114.3)
+		)
+		(stroke
+			(width 0)
+			(type default)
+		)
+	)
+	(wire
+		(pts
+			(xy 101.6 55.88) (xy 101.6 62.23)
+		)
+		(stroke
+			(width 0)
+			(type default)
+		)
+	)
+	(wire
+		(pts
+			(xy 119.38 107.95) (xy 119.38 82.55)
+		)
+		(stroke
+			(width 0)
+			(type default)
+		)
+	)
+	(wire
+		(pts
+			(xy 121.92 105.41) (xy 168.91 105.41)
+		)
+		(stroke
+			(width 0)
+			(type default)
+		)
+	)
+	(wire
+		(pts
+			(xy 121.92 60.96) (xy 121.92 105.41)
+		)
+		(stroke
+			(width 0)
+			(type default)
+		)
+	)
+	(wire
+		(pts
 			(xy 101.6 74.93) (xy 101.6 90.17)
 		)
@@
 	(wire
 		(pts
-			(xy 111.76 74.93) (xy 115.57 74.93)
-		)
-		(stroke
-			(width 0)
-			(type default)
-		)
-	)
-	(wire
-		(pts
-			(xy 111.76 114.3) (xy 180.34 114.3)
-		)
-		(stroke
-			(width 0)
-			(type default)
-		)
-	)
-	(wire
-		(pts
-			(xy 101.6 60.96) (xy 101.6 74.93)
-		)
-		(stroke
-			(width 0)
-			(type default)
-		)
-	)
-	(wire
-		(pts
-			(xy 119.38 107.95) (xy 119.38 82.55)
-		)
-		(stroke
-			(width 0)
-			(type default)
-		)
-	)
-	(wire
-		(pts
-			(xy 121.92 105.41) (xy 168.91 105.41)
-		)
-		(stroke
-			(width 0)
-			(type default)
-		)
-	)
-	(wire
-		(pts
-			(xy 121.92 60.96) (xy 121.92 105.41)
+			(xy 102.87 55.88) (xy 101.6 55.88)
 		)
 		(stroke
@@
 	(wire
 		(pts
+			(xy 113.03 55.88) (xy 113.03 60.96)
+		)
+		(stroke
+			(width 0)
+			(type default)
+		)
+	)
+	(wire
+		(pts
+			(xy 59.69 114.3) (xy 59.69 62.23)
+		)
+		(stroke
+			(width 0)
+			(type default)
+		)
+	)
+	(wire
+		(pts
 			(xy 182.88 82.55) (xy 182.88 123.19)
 		)
@@
 	(wire
 		(pts
-			(xy 111.76 60.96) (xy 121.92 60.96)
+			(xy 59.69 62.23) (xy 101.6 62.23)
 		)
 		(stroke
@@
 	(wire
 		(pts
+			(xy 81.28 153.67) (xy 81.28 167.64)
+		)
+		(stroke
+			(width 0)
+			(type default)
+		)
+	)
+	(wire
+		(pts
 			(xy 176.53 111.76) (xy 176.53 86.36)
 		)
@@
 		(pts
 			(xy 172.72 107.95) (xy 119.38 107.95)
+		)
+		(stroke
+			(width 0)
+			(type default)
+		)
+	)
+	(wire
+		(pts
+			(xy 69.85 114.3) (xy 69.85 153.67)
 		)
 		(stroke
@@
 	)
 	(symbol
+		(lib_id "Switch:SW_Push")
+		(at 64.77 114.3 0)
+		(unit 1)
+		(exclude_from_sim no)
+		(in_bom yes)
+		(on_board yes)
+		(dnp no)
+		(fields_autoplaced yes)
+		(property "Reference" "SW4"
+			(at 64.77 106.68 0)
+			(effects
+				(font
+					(size 1.27 1.27)
+				)
+			)
+		)
+		(property "Value" "SW_Push"
+			(at 64.77 109.22 0)
+			(effects
+				(font
+					(size 1.27 1.27)
+				)
+			)
+		)
+		(property "Footprint" "Button_Switch_Keyboard:SW_Cherry_MX_1.00u_PCB"
+			(at 64.77 109.22 0)
+			(effects
+				(font
+					(size 1.27 1.27)
+				)
+				(hide yes)
+			)
+		)
+		(property "Datasheet" "~"
+			(at 64.77 109.22 0)
+			(effects
+				(font
+					(size 1.27 1.27)
+				)
+				(hide yes)
+			)
+		)
+		(property "Description" "Push button switch, generic, two pins"
+			(at 64.77 114.3 0)
+			(effects
+				(font
+					(size 1.27 1.27)
+				)
+				(hide yes)
+			)
+		)
+		(pin "1"
+		)
+		(pin "2"
+		)
+		(instances
+			(project ""
+				(path "/53fd1076-1de9-405d-b9b9-1c17ddb45294"
+					(reference "SW4")
+					(unit 1)
+				)
+			)
+		)
+	)
+	(symbol
 		(lib_id "power:GND")
 		(at 194.31 87.63 270)
@@
 	(symbol
 		(lib_id "Switch:SW_Push")
-		(at 106.68 60.96 0)
+		(at 107.95 55.88 0)
 		(unit 1)
 		(exclude_from_sim no)
@@
 		(fields_autoplaced yes)
 		(property "Reference" "SW1"
-			(at 106.68 53.34 0)
+			(at 107.95 48.26 0)
 			(effects
 				(font
@@
 		)
 		(property "Value" "SW_Push"
-			(at 106.68 55.88 0)
+			(at 107.95 50.8 0)
 			(effects
 				(font
@@
 		)
 		(property "Footprint" "Button_Switch_Keyboard:SW_Cherry_MX_1.00u_PCB"
-			(at 106.68 55.88 0)
+			(at 107.95 50.8 0)
 			(effects
 				(font
@@
 		)
 		(property "Datasheet" "~"
-			(at 106.68 55.88 0)
+			(at 107.95 50.8 0)
 			(effects
 				(font
@@
 		)
 		(property "Description" "Push button switch, generic, two pins"
-			(at 106.68 60.96 0)
-			(effects
-				(font
+			(at 107.95 55.88 0)
+			(effects
+				(font
